File: sch/mic-test-board/mic-test-pcb.kicad_pcb (KiCad board)
At the start: 4 copper layers, 100 x 100 mm, 126 parts, among them J1 Conn_02x05_Odd_Even, J2 Conn_01x02, U1 NCP163ASN180T1G, U2 SN74LVC2T45DCUR

Commit message: pcb: commit before large routing effort
 - schematic refactor to split preamps to each mic board
 - Mic board and main board are placed
 - no tracks laid
 - critical parts selected
Parts:
- removed C28, C31, C32, C34, C37, C38: 1uF, Capacitor_SMD:C_0603_1608Metric
- removed J1: Conn_02x05_Odd_Even, Connector_PinHeader_2.54mm:PinHeader_2x05_P2.54mm_Vertical
- removed J2: Conn_01x02, Connector_PinHeader_2.54mm:PinHeader_1x02_P2.54mm_Vertical
- removed MK1, MK10, MK11, MK12, MK13, MK14, MK15, MK16, MK2, MK3, MK4, MK5, MK6, MK7, MK8, MK9: ICS-52000, mic-test-board:MIC_ICS-52000
- removed R10, R13, R16, R19, R22, R25: 0R, Resistor_SMD:R_0603_1608Metric
- removed R42, R48: 22.1R, Resistor_SMD:R_0603_1608Metric
- removed R51: 68.1R, Resistor_SMD:R_0603_1608Metric
- added C100: 10nF, Capacitor_SMD:C_0603_1608Metric, F.Cu at (150.0, 124.7)
- added C101: 10nF, Capacitor_SMD:C_0603_1608Metric, F.Cu at (150.3, 129.3)
- added C104: 10nF, Capacitor_SMD:C_0603_1608Metric, F.Cu at (149.5, 127.0)
- added C106: 10nF, Capacitor_SMD:C_0603_1608Metric, F.Cu at (150.1, 115.3)
- added C107: 10nF, Capacitor_SMD:C_0603_1608Metric, F.Cu at (150.3, 119.9)
- added C110: 10nF, Capacitor_SMD:C_0603_1608Metric, F.Cu at (149.5, 117.6)
- added C112: 10nF, Capacitor_SMD:C_0603_1608Metric, F.Cu at (127.8, 135.9)
- added C113: 10nF, Capacitor_SMD:C_0603_1608Metric, F.Cu at (123.2, 136.1)
- added C116: 10nF, Capacitor_SMD:C_0603_1608Metric, F.Cu at (125.5, 135.4)
- added C118: 10nF, Capacitor_SMD:C_0603_1608Metric, F.Cu at (118.2, 135.9)
- added C119: 10nF, Capacitor_SMD:C_0603_1608Metric, F.Cu at (113.6, 136.1)
- added C122: 10nF, Capacitor_SMD:C_0603_1608Metric, F.Cu at (115.9, 135.4)
- added C124: 10nF, Capacitor_SMD:C_0603_1608Metric, F.Cu at (109.0, 124.5)
- added C125: 10nF, Capacitor_SMD:C_0603_1608Metric, F.Cu at (108.7, 119.9)
- added C128: 10nF, Capacitor_SMD:C_0603_1608Metric, F.Cu at (109.5, 122.2)
- added C130: 10nF, Capacitor_SMD:C_0603_1608Metric, F.Cu at (109.0, 115.1)
- added C131: 10nF, Capacitor_SMD:C_0603_1608Metric, F.Cu at (108.7, 110.5)
- added C134: 10nF, Capacitor_SMD:C_0603_1608Metric, F.Cu at (109.5, 112.8)
- added C186: 10nF, Capacitor_SMD:C_0603_1608Metric, F.Cu at (108.7, 78.7)
- added C187: 10nF, Capacitor_SMD:C_0603_1608Metric, F.Cu at (109.4, 80.9)
- added C201: 0.1uF, Capacitor_SMD:C_0603_1608Metric, F.Cu at (248.4, 85.1)
- added C208: 0.1uF, Capacitor_SMD:C_0603_1608Metric, F.Cu at (120.4, 115.8)
- added C209: 0.1uF, Capacitor_SMD:C_0603_1608Metric, F.Cu at (140.7, 95.8)
- added C210: 0.1uF, Capacitor_SMD:C_0603_1608Metric, F.Cu at (140.7, 115.6)
- added C211: 0.1uF, Capacitor_SMD:C_0603_1608Metric, F.Cu at (120.9, 96.4)
- added C41: 10nF, Capacitor_SMD:C_0603_1608Metric, F.Cu at (122.2, 72.4)
- added C42: 10nF, Capacitor_SMD:C_0603_1608Metric, F.Cu at (126.7, 72.1)
- added C45: 10nF, Capacitor_SMD:C_0603_1608Metric, F.Cu at (124.5, 72.9)
- added C47: 10nF, Capacitor_SMD:C_0603_1608Metric, F.Cu at (131.8, 72.4)
- added C48: 10nF, Capacitor_SMD:C_0603_1608Metric, F.Cu at (136.4, 72.1)
- added C51: 10nF, Capacitor_SMD:C_0603_1608Metric, F.Cu at (134.1, 72.9)
- added C53: 10nF, Capacitor_SMD:C_0603_1608Metric, F.Cu at (149.3, 78.7)
- added C54: 10nF, Capacitor_SMD:C_0603_1608Metric, F.Cu at (149.6, 83.3)
- added C57: 10nF, Capacitor_SMD:C_0603_1608Metric, F.Cu at (148.8, 81.0)
- added C59: 1uF, Capacitor_SMD:C_0603_1608Metric, F.Cu at (168.4, 89.5)
- added C60: 1uF, Capacitor_SMD:C_0603_1608Metric, F.Cu at (170.7, 88.7)
- added C61: 1uF, Capacitor_SMD:C_0603_1608Metric, F.Cu at (175.0, 109.7)
- added C62: 1uF, Capacitor_SMD:C_0603_1608Metric, F.Cu at (172.7, 110.5)
- added C63: 1uF, Capacitor_SMD:C_0603_1608Metric, F.Cu at (175.0, 119.8)
- added C64: 1uF, Capacitor_SMD:C_0603_1608Metric, F.Cu at (172.7, 120.6)
- added C65: 10nF, Capacitor_SMD:C_0603_1608Metric, F.Cu at (149.3, 88.1)
- added C66: 10nF, Capacitor_SMD:C_0603_1608Metric, F.Cu at (149.6, 92.6)
- added C67: 1uF, Capacitor_SMD:C_0603_1608Metric, F.Cu at (140.7, 117.1)
- added C68: 0.1uF, Capacitor_SMD:C_0603_1608Metric, F.Cu at (140.7, 118.6)
- added C69: 1uF, Capacitor_SMD:C_0603_1608Metric, F.Cu at (120.4, 118.9)
- added C70: 0.1uF, Capacitor_SMD:C_0603_1608Metric, F.Cu at (120.4, 117.3)
- added C71: 1uF, Capacitor_SMD:C_0603_1608Metric, F.Cu at (133.6, 125.5)
- added C72: 0.1uF, Capacitor_SMD:C_0603_1608Metric, F.Cu at (132.1, 125.5)
- added C73: 1uF, Capacitor_SMD:C_0603_1608Metric, F.Cu at (129.0, 125.5)
- added C74: 0.1uF, Capacitor_SMD:C_0603_1608Metric, F.Cu at (127.5, 125.5)
- added C75: 1uF, Capacitor_SMD:C_0603_1608Metric, F.Cu at (120.4, 113.5)
- added C76: 0.1uF, Capacitor_SMD:C_0603_1608Metric, F.Cu at (120.4, 112.0)
- added C77: 1uF, Capacitor_SMD:C_0603_1608Metric, F.Cu at (120.4, 110.5)
- added C78: 0.1uF, Capacitor_SMD:C_0603_1608Metric, F.Cu at (120.4, 109.0)
- added C79: 1uF, Capacitor_SMD:C_0603_1608Metric, F.Cu at (136.6, 125.5)
- added C80: 0.1uF, Capacitor_SMD:C_0603_1608Metric, F.Cu at (135.1, 125.5)
- added C81: 1uF, Capacitor_SMD:C_0603_1608Metric, F.Cu at (126.0, 125.5)
- added C82: 0.1uF, Capacitor_SMD:C_0603_1608Metric, F.Cu at (124.4, 125.5)
- added C83: 0.1uF, Capacitor_SMD:C_0603_1608Metric, F.Cu at (130.5, 129.3)
- added C86: 10nF, Capacitor_SMD:C_0603_1608Metric, F.Cu at (148.8, 90.3)
- added C88: 10nF, Capacitor_SMD:C_0603_1608Metric, F.Cu at (137.5, 135.9)
- added C89: 10nF, Capacitor_SMD:C_0603_1608Metric, F.Cu at (132.9, 136.1)
- added C92: 10nF, Capacitor_SMD:C_0603_1608Metric, F.Cu at (135.2, 135.4)
- added C94: 10nF, Capacitor_SMD:C_0603_1608Metric, F.Cu at (150.0, 134.0)
- added C95: 10nF, Capacitor_SMD:C_0603_1608Metric, F.Cu at (150.3, 138.6)
- added C98: 10nF, Capacitor_SMD:C_0603_1608Metric, F.Cu at (149.5, 136.3)
- added D10: LED_Small_Filled, LED_SMD:LED_0805_2012Metric, F.Cu at (240.9, 135.6)
- added D2: LED_Small_Filled, LED_SMD:LED_0805_2012Metric, F.Cu at (169.2, 108.5)
- added D3: LED_Small_Filled, LED_SMD:LED_0805_2012Metric, F.Cu at (240.9, 113.0)
- added D4: LED_Small_Filled, LED_SMD:LED_0805_2012Metric, F.Cu at (240.9, 116.3)
- added D5: LED_Small_Filled, LED_SMD:LED_0805_2012Metric, F.Cu at (241.0, 119.6)
- added D6: LED_Small_Filled, LED_SMD:LED_0805_2012Metric, F.Cu at (240.9, 122.4)
- added D7: LED_Small_Filled, LED_SMD:LED_0805_2012Metric, F.Cu at (240.9, 125.7)
- added D8: LED_Small_Filled, LED_SMD:LED_0805_2012Metric, F.Cu at (240.9, 129.0)
- added D9: LED_Small_Filled, LED_SMD:LED_0805_2012Metric, F.Cu at (240.9, 132.3)
- added J11: Conn_01x04, mic-test-board:Molex_PicoBlade_53047-0510_1x05_P1.25mm_Vertical, F.Cu at (102.9, 96.5)
- added J13: Conn_01x04, mic-test-board:Molex_PicoBlade_53047-0510_1x05_P1.25mm_Vertical, F.Cu at (127.8, 66.3)
- added J15: Conn_01x04, mic-test-board:Molex_PicoBlade_53047-0510_1x05_P1.25mm_Vertical, F.Cu at (137.4, 66.3)
- added J17: Conn_01x04, mic-test-board:Molex_PicoBlade_53047-0510_1x05_P1.25mm_Vertical, F.Cu at (155.4, 84.3)
- added J19: Conn_01x04, mic-test-board:Molex_PicoBlade_53047-0510_1x05_P1.25mm_Vertical, F.Cu at (155.4, 93.6)
- added J21: Conn_01x04, mic-test-board:Molex_PicoBlade_53047-0510_1x05_P1.25mm_Vertical, F.Cu at (131.9, 142.0)
- added J23: Conn_01x04, mic-test-board:Molex_PicoBlade_53047-0510_1x05_P1.25mm_Vertical, F.Cu at (156.1, 139.6)
- added J25: Conn_01x04, mic-test-board:Molex_PicoBlade_53047-0510_1x05_P1.25mm_Vertical, F.Cu at (156.1, 130.3)
- added J27: Conn_01x04, mic-test-board:Molex_PicoBlade_53047-0510_1x05_P1.25mm_Vertical, F.Cu at (156.1, 120.9)
- added J29: Conn_01x04, mic-test-board:Molex_PicoBlade_53047-0510_1x05_P1.25mm_Vertical, F.Cu at (122.2, 142.0)
- added J3: Conn_01x03, Connector_PinHeader_2.54mm:PinHeader_1x02_P2.54mm_Vertical, F.Cu at (208.3, 65.8)
- added J31: Conn_01x04, mic-test-board:Molex_PicoBlade_53047-0510_1x05_P1.25mm_Vertical, F.Cu at (112.6, 142.0)
- added J33: Conn_01x04, mic-test-board:Molex_PicoBlade_53047-0510_1x05_P1.25mm_Vertical, F.Cu at (102.9, 118.9)
- added J35: Conn_01x04, mic-test-board:Molex_PicoBlade_53047-0510_1x05_P1.25mm_Vertical, F.Cu at (102.9, 109.5)
- added J4: Conn_01x03, TerminalBlock_Phoenix:TerminalBlock_Phoenix_MKDS-1,5-2_1x02_P5.00mm_Horizontal, F.Cu at (177.9, 103.6)
- added J7: Conn_01x04, mic-test-board:Molex_PicoBlade_53047-0510_1x05_P1.25mm_Vertical, F.Cu at (102.8, 68.2)
- added J8: Conn_01x04, mic-test-board:Molex_PicoBlade_53047-0510_1x05_P1.25mm_Vertical, F.Cu at (102.8, 77.6)
- added J9: Conn_01x04, mic-test-board:Molex_PicoBlade_53047-0510_1x05_P1.25mm_Vertical, F.Cu at (102.8, 87.0)
- added JP18: SolderJumper_3_Open, Jumper:SolderJumper-3_P1.3mm_Open_RoundedPad1.0x1.5mm_NumberLabels, F.Cu at (169.4, 117.3)
- added JP20: SolderJumper_2_Bridged, Jumper:SolderJumper-2_P1.3mm_Bridged_Pad1.0x1.5mm, F.Cu at (188.9, 38.1)
- added JP21: SolderJumper_2_Bridged, Jumper:SolderJumper-2_P1.3mm_Bridged_Pad1.0x1.5mm, F.Cu at (189.5, 34.0)
- added R101: 0R, Resistor_SMD:R_0603_1608Metric, F.Cu at (107.1, 109.0)
- added R102: 33R, Resistor_SMD:R_0603_1608Metric, F.Cu at (107.2, 113.6)
- added R105: 33R, Resistor_SMD:R_0603_1608Metric, F.Cu at (107.2, 112.1)
- added R118: 0R, Resistor_SMD:R_0603_1608Metric, F.Cu at (250.7, 92.2)
- added R119: 0R, Resistor_SMD:R_0603_1608Metric, F.Cu at (254.0, 92.2)
- added R120: 0R, Resistor_SMD:R_0603_1608Metric, F.Cu at (255.8, 86.9)
- added R135: 470R, Resistor_SMD:R_0603_1608Metric, F.Cu at (237.5, 113.0)
- added R136: 470R, Resistor_SMD:R_0603_1608Metric, F.Cu at (237.5, 116.3)
- added R137: 470R, Resistor_SMD:R_0603_1608Metric, F.Cu at (237.6, 119.6)
- added R138: 470R, Resistor_SMD:R_0603_1608Metric, F.Cu at (237.5, 122.4)
- added R139: 470R, Resistor_SMD:R_0603_1608Metric, F.Cu at (237.5, 125.7)
- added R14: 0R, Resistor_SMD:R_0603_1608Metric, F.Cu at (107.1, 96.0)
- added R140: 470R, Resistor_SMD:R_0603_1608Metric, F.Cu at (237.5, 129.0)
- added R141: 470R, Resistor_SMD:R_0603_1608Metric, F.Cu at (237.5, 132.3)
- added R142: 470R, Resistor_SMD:R_0603_1608Metric, F.Cu at (237.3, 135.6)
- added R20: 0R, Resistor_SMD:R_0603_1608Metric, F.Cu at (128.3, 70.5)
- added R223: 33R, Resistor_SMD:R_0603_1608Metric, F.Cu at (107.2, 70.8)
- added R238: 0R, Resistor_SMD:R_0603_1608Metric, F.Cu at (107.1, 67.7)
- added R26: 0R, Resistor_SMD:R_0603_1608Metric, F.Cu at (177.3, 111.7)
- added R29: 100k, Resistor_SMD:R_0603_1608Metric, F.Cu at (168.4, 92.5)
- added R32: 0R, Resistor_SMD:R_0603_1608Metric, F.Cu at (177.3, 121.9)
- added R35: 0R, Resistor_SMD:R_0603_1608Metric, F.Cu at (154.2, 104.6)
- added R38: 0R, Resistor_SMD:R_0603_1608Metric, F.Cu at (150.5, 109.2)
- added R54: 33R, Resistor_SMD:R_0603_1608Metric, F.Cu at (151.1, 89.6)
- added R57: 33R, Resistor_SMD:R_0603_1608Metric, F.Cu at (151.1, 91.1)
- added R59: 0R, Resistor_SMD:R_0603_1608Metric, F.Cu at (131.4, 137.7)
- added R60: 33R, Resistor_SMD:R_0603_1608Metric, F.Cu at (136.0, 137.7)
- added R63: 33R, Resistor_SMD:R_0603_1608Metric, F.Cu at (134.4, 137.7)
- added R65: 0R, Resistor_SMD:R_0603_1608Metric, F.Cu at (151.9, 140.1)
- added R66: 33R, Resistor_SMD:R_0603_1608Metric, F.Cu at (151.8, 135.6)
- added R69: 33R, Resistor_SMD:R_0603_1608Metric, F.Cu at (151.8, 137.1)
- added R71: 0R, Resistor_SMD:R_0603_1608Metric, F.Cu at (151.9, 130.8)
- added R72: 33R, Resistor_SMD:R_0603_1608Metric, F.Cu at (151.8, 126.2)
- added R75: 33R, Resistor_SMD:R_0603_1608Metric, F.Cu at (151.8, 127.8)
- added R77: 0R, Resistor_SMD:R_0603_1608Metric, F.Cu at (151.9, 121.4)
- added R78: 33R, Resistor_SMD:R_0603_1608Metric, F.Cu at (151.8, 116.8)
- added R81: 33R, Resistor_SMD:R_0603_1608Metric, F.Cu at (151.8, 118.4)
- added R83: 0R, Resistor_SMD:R_0603_1608Metric, F.Cu at (121.7, 137.7)
- added R84: 33R, Resistor_SMD:R_0603_1608Metric, F.Cu at (126.2, 137.7)
- added R87: 33R, Resistor_SMD:R_0603_1608Metric, F.Cu at (124.7, 137.7)
- added R89: 0R, Resistor_SMD:R_0603_1608Metric, F.Cu at (112.1, 137.7)
- added R90: 33R, Resistor_SMD:R_0603_1608Metric, F.Cu at (116.7, 137.7)
- added R93: 33R, Resistor_SMD:R_0603_1608Metric, F.Cu at (115.1, 137.7)
- added R95: 0R, Resistor_SMD:R_0603_1608Metric, F.Cu at (107.1, 118.4)
- added R96: 33R, Resistor_SMD:R_0603_1608Metric, F.Cu at (107.2, 122.9)
- added R99: 33R, Resistor_SMD:R_0603_1608Metric, F.Cu at (107.2, 121.4)
- added SW1: SW_Push, Button_Switch_SMD:SW_SPST_CK_RS282G05A3, F.Cu at (62.2, 48.0)
- added SW2: SW_Push, Button_Switch_SMD:SW_SPST_CK_RS282G05A3, F.Cu at (62.2, 51.0)
- added TP10: TestPoint, TestPoint:TestPoint_Pad_D1.0mm, F.Cu at (175.0, 114.3)
- added TP11: TestPoint, TestPoint:TestPoint_Pad_D1.0mm, F.Cu at (177.5, 119.1)
- added TP12: TestPoint, TestPoint:TestPoint_Pad_D1.0mm, F.Cu at (174.5, 124.4)
- added TP13: TestPoint, TestPoint:TestPoint_Pad_D1.0mm, F.Cu at (51.6, 86.9)
- added TP14: TestPoint, TestPoint:TestPoint_Pad_D1.0mm, F.Cu at (51.6, 89.9)
- added TP15: TestPoint, TestPoint:TestPoint_Pad_D1.0mm, F.Cu at (154.2, 109.0)
- added TP16: TestPoint, TestPoint:TestPoint_Pad_D1.0mm, F.Cu at (147.8, 104.1)
- added TP17: TestPoint, TestPoint:TestPoint_Pad_D1.0mm, F.Cu at (147.8, 109.2)
- added TP18: TestPoint, TestPoint:TestPoint_Pad_D1.0mm, F.Cu at (207.2, 96.1)
- added TP19: TestPoint, TestPoint:TestPoint_Pad_D1.0mm, F.Cu at (207.2, 93.1)
- added TP20: TestPoint, TestPoint:TestPoint_Pad_D1.0mm, F.Cu at (207.2, 90.0)
- added TP21: TestPoint, TestPoint:TestPoint_Pad_D1.0mm, F.Cu at (207.2, 87.0)
- added TP22: TestPoint, TestPoint:TestPoint_Pad_D1.0mm, F.Cu at (207.2, 83.9)
- added TP23: TestPoint, TestPoint:TestPoint_Pad_D1.0mm, F.Cu at (247.1, 93.2)
- added TP24: TestPoint, TestPoint:TestPoint_Pad_D1.0mm, F.Cu at (257.3, 91.4)
- added TP25: TestPoint, TestPoint:TestPoint_Pad_D1.0mm, F.Cu at (255.5, 88.9)
- added TP26: TestPoint, TestPoint:TestPoint_Pad_D1.0mm, F.Cu at (247.1, 90.9)
- added TP27: TestPoint, TestPoint:TestPoint_Pad_D1.0mm, F.Cu at (242.3, 88.4)
- added TP28: TestPoint, TestPoint:TestPoint_Pad_D1.0mm, F.Cu at (256.5, 98.8)
- added TP29: TestPoint, TestPoint:TestPoint_Pad_D1.0mm, F.Cu at (255.3, 84.6)
- added TP30: TestPoint, TestPoint:TestPoint_Pad_D1.0mm, F.Cu at (174.2, 45.7)
- added TP31: TestPoint, TestPoint:TestPoint_Pad_D1.0mm, F.Cu at (174.2, 48.8)
- added TP32: TestPoint, TestPoint:TestPoint_Pad_D1.0mm, F.Cu at (174.2, 51.8)
- added TP33: TestPoint, TestPoint:TestPoint_Pad_D1.0mm, F.Cu at (177.3, 39.6)
- added TP34: TestPoint, TestPoint:TestPoint_Pad_D1.0mm, F.Cu at (177.3, 42.7)
- added TP35: TestPoint, TestPoint:TestPoint_Pad_D1.0mm, F.Cu at (177.3, 45.7)
- added TP36: Hole_1.5mm, TestPoint:TestPoint_THTPad_D1.5mm_Drill0.7mm, F.Cu at (113.3, 69.9)
- added TP37: TestPoint, TestPoint:TestPoint_Pad_D1.0mm, F.Cu at (161.3, 99.3)
- added TP7: TestPoint, TestPoint:TestPoint_Pad_D1.0mm, F.Cu at (170.4, 93.3)
- added TP8: TestPoint, TestPoint:TestPoint_Pad_D1.0mm, F.Cu at (177.5, 109.0)
- added TP9: TestPoint, TestPoint:TestPoint_Pad_D1.0mm, F.Cu at (173.2, 88.0)
- added U22: LP5912-5.0DRV, Package_SON:WSON-6-1EP_2x2mm_P0.65mm_EP1x1.6mm_ThermalVias, F.Cu at (170.7, 90.9)
- added U23: LP5912-3.3DRV, Package_SON:WSON-6-1EP_2x2mm_P0.65mm_EP1x1.6mm_ThermalVias, F.Cu at (175.0, 122.0)
- added U24: LP5912-3.3DRV, Package_SON:WSON-6-1EP_2x2mm_P0.65mm_EP1x1.6mm_ThermalVias, F.Cu at (175.1, 111.9)
- added U3: MAX6070BAUT33+T, Package_TO_SOT_SMD:SOT-23-6, F.Cu at (164.3, 102.2)
- added U34: SN74LVC126ARGYR, mic-test-board:IC_SN74AUC08RGYRG4, F.Cu at (251.7, 87.6)
- added U5: NUCLEO144-H743ZI, mic-test-board:ST_Morpho_Connector_144_STLink_SMD_Headers_BottomMount, F.Cu at (221.8, 64.5)
- added U6: AD7768BSTZ, Package_QFP:LQFP-64_10x10mm_P0.5mm, F.Cu at (130.5, 115.4)
- added X1: KC3225Z32.7680C1KX00, Oscillator:Oscillator_SMD_SeikoEpson_SG210-4Pin_2.5x2.0mm, F.Cu at (156.4, 104.9)
- C1, C12, C15, C16, C3, C5, C7, C9: value 0.1uF -> 1uF
- C18, C20: value 22pF -> 10nF
- C19: value 22pF -> 1uF
- C22, C25: value 1uF -> 0.1uF
- C23: value 22pF -> 0.1uF
- C26, C27, C29, C30, C33, C35, C36, C39: value 1uF -> 10nF
- JP1, JP2: value SolderJumper_2_Open -> SolderJumper_3_Open; footprint Jumper:SolderJumper-2_P1.3mm_Open_TrianglePad1.0x1.5mm -> Jumper:SolderJumper-3_P1.3mm_Open_RoundedPad1.0x1.5mm_NumberLabels
- JP10, JP11, JP12, JP13, JP14, JP15, JP3, JP4, JP5, JP6, JP7, JP8, JP9: value SolderJumper_2_Open -> SolderJumper_2_Bridged; footprint Jumper:SolderJumper-2_P1.3mm_Open_TrianglePad1.0x1.5mm -> Jumper:SolderJumper-2_P1.3mm_Bridged_Pad1.0x1.5mm
- JP16, JP17: value SolderJumper_3_Open -> SolderJumper_2_Bridged; footprint Jumper:SolderJumper-3_P2.0mm_Open_TrianglePad1.0x1.5mm_NumberLabels -> Jumper:SolderJumper-2_P1.3mm_Bridged_Pad1.0x1.5mm
- R1: value 68.1R -> 49.9R
- R12, R15, R18, R21, R24, R30, R6, R9: value 22.1R -> 33R
- R2, R27, R39, R45: value 22.1R -> 0R
- R31, R34: value 0R -> 100k
- R33: value 22.1R -> 470R
- R36: value 22.1R -> 100k
- R4: value 0R -> 470R
- R40: value 0R -> 49.9R
- R43, R46, R49, R7: value 0R -> 33R
- R5: value 68.1R -> 33R
- R50, R52: value 68.1R -> 49.9k
- R53: value 68.1R -> 0R
- R8: value 180R -> 0R
- TP1, TP3, TP5, TP6: footprint TestPoint:TestPoint_Pad_D1.5mm -> TestPoint:TestPoint_Pad_D1.0mm
- TP2: value (none) -> TestPoint; footprint TestPoint:TestPoint_Pad_D1.5mm -> TestPoint:TestPoint_Pad_D1.0mm
- TP4: value (none) -> Hole_1.5mm; footprint TestPoint:TestPoint_Pad_D1.5mm -> TestPoint:TestPoint_THTPad_D1.5mm_Drill0.7mm
- U1: value NCP163ASN180T1G -> LMK1C1102; footprint Package_TO_SOT_SMD:SOT-23-5 -> Package_SON:WSON-8-1EP_2x2mm_P0.5mm_EP0.9x1.6mm
- U2: value SN74LVC2T45DCUR -> AD7768BSTZ; footprint Package_SO:VSSOP-8_2.4x2.1mm_P0.5mm -> Package_QFP:LQFP-64_10x10mm_P0.5mm
- moved JP9 140.9 mm to (244.3, 116.3), turned to 180 degrees
- moved JP10 130.3 mm to (244.3, 113.0), turned to 180 degrees
- moved JP15 123.2 mm to (188.7, 30.2)
- moved JP8 120.4 mm to (244.4, 119.6), turned to 180 degrees
- moved JP7 117.3 mm to (244.4, 122.4), turned to 180 degrees
- moved TP3 113.0 mm to (51.3, 74.1)
- moved JP6 111.3 mm to (244.4, 125.7), turned to 180 degrees
- moved TP6 111.2 mm to (51.6, 83.8), turned to 0 degrees
- moved JP14 110.6 mm to (180.8, 26.9), turned to 0 degrees
- moved JP11 102.5 mm to (252.2, 95.8), turned to 90 degrees
- moved TP5 102.3 mm to (51.6, 80.8)
- moved H1 99.9 mm to (27.0, 60.7)
- moved H2 99.9 mm to (79.1, 61.0)
- moved H3 99.9 mm to (53.1, 105.9)
- moved JP5 94.8 mm to (244.5, 129.0)
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Connections:
- C1 pad 1: VDD -> +5VA
- C10 pad 1: VDD -> +3.3V
- C11 pad 1: VDD -> /ADC1 AD7768/V_{OCM}
- C12 pad 1: VDD -> +5VA
- C13 pad 1: VDD -> Net-(U3-FILTER)
- C14 pad 1: VDD -> /V_{REF}
- C15 pad 1: VDD -> /V_{REF}
- C16 pad 1: VDD -> /ADC1 AD7768/DREGCAP
- C17 pad 1: VDD -> /ADC1 AD7768/DREGCAP
- C18 pad 1: Net-(C18-Pad1) -> GND
- C18 pad 2: GND -> /ADC1 AD7768/AIN1+
- C19 pad 1: Net-(C19-Pad1) -> /ADC1 AD7768/REGCAPA
- C2 pad 1: VDD -> +5VA
- C20 pad 1: Net-(C20-Pad1) -> GND
- C20 pad 2: GND -> /ADC1 AD7768/AIN0+
- C21 pad 1: Net-(J2-Pin_1) -> +3.3V
- C22 pad 1: VDD -> +3.3V
- C23 pad 1: Net-(C23-Pad1) -> /ADC1 AD7768/REGCAPA
- C24 pad 1: VDD -> /ADC1 AD7768/REGCAPB
- C25 pad 1: VDD -> /ADC1 AD7768/REGCAPB
- C26 pad 1: VDD -> /ADC1 AD7768/AIN0-
- C27 pad 1: VDD -> /ADC1 AD7768/AIN0+
- C27 pad 2: GND -> /ADC1 AD7768/AIN0-
- C29 pad 1: VDD -> GND
- C29 pad 2: GND -> /ADC1 AD7768/AIN2+
- C3 pad 1: VDD -> +5VA
- C30 pad 1: VDD -> /ADC1 AD7768/AIN2-
- C33 pad 1: VDD -> /ADC1 AD7768/AIN2+
- C33 pad 2: GND -> /ADC1 AD7768/AIN2-
- C35 pad 1: VDD -> GND
- C35 pad 2: GND -> /ADC1 AD7768/AIN3+
- C36 pad 1: VDD -> /ADC1 AD7768/AIN3-
- C39 pad 1: VDD -> /ADC1 AD7768/AIN3+
- C39 pad 2: GND -> /ADC1 AD7768/AIN3-
- C4 pad 1: VDD -> +5VA
- C5 pad 1: VDD -> +3.3V
- C6 pad 1: VDD -> +3.3V
- C7 pad 1: VDD -> +3.3V
- C8 pad 1: VDD -> +3.3V
- C9 pad 1: VDD -> +3.3V
- JP1 pad 1: /Mic1/WSO -> GND
- JP1 pad 2: /Mic2/WS -> Net-(JP1-C)
- JP10 pad 1: /Mic10/WSO -> /uController/LED8_uC
- JP10 pad 2: /Mic11/WS -> /uController/LED8
- JP11 pad 1: /Mic11/WSO -> +3.3V
- JP11 pad 2: /Mic12/WS -> Net-(JP11-B)
- JP12 pad 1: /Mic12/WSO -> +3.3V
- JP12 pad 2: /Mic13/WS -> Net-(JP12-B)
- JP13 pad 1: /Mic13/WSO -> /DRDY
- JP13 pad 2: /Mic14/WS -> Net-(JP13-B)
- JP14 pad 1: /Mic14/WSO -> /ADC1 AD7768/~{START}
- JP14 pad 2: /Mic15/WS -> /uController/GPIO_~{START}_uC
- JP15 pad 1: /Mic15/WSO -> /SPI1_~{CS1}
- JP15 pad 2: /Mic16/WS -> /uController/SPI1_~{CS1}_uC
- JP16 pad 1: Net-(JP16-A) -> /SPI1_~{CS2}
- JP16 pad 2: /Mic1/SCK -> /uController/SPI1_~{CS2}_uC
- JP17 pad 1: Net-(JP17-A) -> /SPI1_SCLK
- JP17 pad 2: /Mic1/SD -> /uController/SPI1_SCLK_uC
- JP2 pad 1: /Mic2/WSO -> GND
- JP2 pad 2: /Mic3/WS -> Net-(JP2-C)
- JP3 pad 1: /Mic3/WSO -> /uController/LED1_uC
- JP3 pad 2: /Mic4/WS -> /uController/LED1
- JP4 pad 1: /Mic4/WSO -> /uController/LED2_uC
- JP4 pad 2: /Mic5/WS -> /uController/LED2
- JP5 pad 1: /Mic5/WSO -> /uController/LED3_uC
- JP5 pad 2: /Mic6/WS -> /uController/LED3
- JP6 pad 1: /Mic6/WSO -> /uController/LED4_uC
- JP6 pad 2: /Mic7/WS -> /uController/LED4
- JP7 pad 1: /Mic7/WSO -> /uController/LED5_uC
- JP7 pad 2: /Mic8/WS -> /uController/LED5
- JP8 pad 1: /Mic8/WSO -> /uController/LED6_uC
- JP8 pad 2: /Mic9/WS -> /uController/LED6
- JP9 pad 1: /Mic9/WSO -> /uController/LED7_uC
- JP9 pad 2: /Mic10/WS -> /uController/LED7
- R1 pad 1: /Mic1/SCK -> Net-(U2-VCM)
- R1 pad 2: Net-(C23-Pad1) -> /ADC1 AD7768/V_{OCM}
- R12 pad 2: /Mic1/SD -> /ADC1 AD7768/AIN2-
- R15 pad 2: /Mic1/SD -> /ADC1 AD7768/AIN3+
- R18 pad 2: /Mic1/SD -> /ADC1 AD7768/AIN3-
- R2 pad 1: Net-(MK1-SD) -> GND
- R2 pad 2: /Mic1/SD -> Net-(U2-CLK_SEL)
- R21 pad 2: /Mic1/SD -> /ADC1 AD7768/AIN4+
- R24 pad 2: /Mic1/SD -> /ADC1 AD7768/AIN4-
- R27 pad 1: Net-(MK9-SD) -> GND
- R27 pad 2: /Mic1/SD -> Net-(J15-Pin_1)
- R28 pad 1: /Mic9/WS -> /V_{IN}
- R28 pad 2: /Mic9/WSO -> Net-(U22-EN)
- R3 pad 1: /WS -> GND
- R3 pad 2: /Mic1/WSO -> Net-(J8-Pin_1)
- R30 pad 2: /Mic1/SD -> /ADC1 AD7768/AIN5+
- R31 pad 1: /Mic13/WS -> Net-(U24-PG)
- R31 pad 2: /Mic13/WSO -> +3.3V
- R33 pad 1: Net-(MK15-SD) -> +3.3V
- R33 pad 2: /Mic1/SD -> Net-(D2-A)
- R34 pad 1: /Mic15/WS -> Net-(U23-PG)
- R34 pad 2: /Mic15/WSO -> Net-(JP18-A)
- R36 pad 1: Net-(MK12-SD) -> Net-(U1-1G/Enable)
- R36 pad 2: /Mic1/SD -> +3.3V
- R37 pad 1: /Mic12/WS -> Net-(U1-Y0)
- R37 pad 2: /Mic12/WSO -> /MCLK_1
- R39 pad 1: Net-(MK14-SD) -> GND
- R39 pad 2: /Mic1/SD -> Net-(U6-CLK_SEL)
- R4 pad 1: VDD -> +5VA
- R40 pad 1: /Mic14/WS -> Net-(U6-VCM)
- R40 pad 2: /Mic14/WSO -> /ADC2 AD7769/V_{OCM}
- R43 pad 1: /Mic10/WS -> Net-(J15-Pin_3)
- R43 pad 2: /Mic10/WSO -> /ADC1 AD7768/AIN5-
- R45 pad 1: Net-(MK16-SD) -> GND
- R45 pad 2: /Mic1/SD -> Net-(J17-Pin_1)
- R46 pad 1: /Mic16/WS -> Net-(J17-Pin_4)
- R46 pad 2: /Mic16/WSO -> /ADC1 AD7768/AIN6+
- R49 pad 1: /Mic11/WS -> Net-(J17-Pin_3)
- R49 pad 2: /Mic11/WSO -> /ADC1 AD7768/AIN6-
- R5 pad 1: /Mic1/SD -> Net-(J8-Pin_4)
- R5 pad 2: GND -> /ADC1 AD7768/AIN1+
- R50 pad 1: /SCK -> /uController/~{PButton1}
- R50 pad 2: Net-(C18-Pad1) -> +3.3V
- R52 pad 1: /WS -> /uController/~{PButton2}
- R52 pad 2: Net-(C20-Pad1) -> +3.3V
- R53 pad 1: Net-(JP16-A) -> GND
- R53 pad 2: Net-(U2-B1) -> Net-(J19-Pin_1)
- R6 pad 2: /Mic1/SD -> /ADC1 AD7768/AIN1-
- R7 pad 1: /Mic2/WS -> Net-(J7-Pin_4)
- R7 pad 2: /Mic2/WSO -> /ADC1 AD7768/AIN0+
- R8 pad 1: /Mic1/SCK -> GND
- R8 pad 2: GND -> Net-(J9-Pin_1)
- R9 pad 2: /Mic1/SD -> /ADC1 AD7768/AIN2+
- TP1 pad 1: /Mic16/WSO -> Net-(U2-MODE0/GPIO0)
- TP2 pad 1: /SD -> Net-(U6-~{RESET})
- TP3 pad 1: /SCK -> Net-(U2-~{RESET})
- TP4 pad 1: /WS -> /ADC1 AD7768/AIN0+
- TP5 pad 1: Net-(JP16-A) -> Net-(U2-MODE1/GPIO1)
- TP6 pad 1: /Mic1/SD -> Net-(U2-MODE2/GPIO2)
- U1 pad 1: Net-(J2-Pin_1) -> Net-(U1-CLKIN)
- U1 pad 2: GND -> Net-(U1-1G/Enable)
- U1 pad 3: Net-(J2-Pin_1) -> Net-(U1-Y0)
- U1 pad 4: unconnected-(U1-NC-Pad4) -> GND
- U1 pad 5: VDD -> (no net)
- U2 pad 1: VDD -> /ADC1 AD7768/AIN1-
- U2 pad 2: /SCK -> /ADC1 AD7768/AIN1+
- U2 pad 3: Net-(JP17-A) -> GND
- U2 pad 4: GND -> +5VA
- U2 pad 5: VDD -> GND
- U2 pad 6: /SD -> /V_{REF}
- U2 pad 7: Net-(U2-B1) -> /ADC1 AD7768/AIN2-
- U2 pad 8: VDD -> /ADC1 AD7768/AIN2+
Routing:
- net /Mic1/SCK: track 425.1 -> 0.00 mm
- net /Mic1/SD: track 407.5 -> 0.00 mm
- net GND: track 122.0 -> 0.00 mm, vias 146 -> 0
- net VDD: track 106.1 -> 0.00 mm, vias 20 -> 0
- net /WS: track 42.2 -> 0.00 mm, vias 1 -> 0
- net /Mic9/WS: track 39.8 -> 0.00 mm, vias 2 -> 0
- net /Mic15/WS: track 34.8 -> 0.00 mm
- net /SCK: track 34.0 -> 0.00 mm, vias 2 -> 0
- net /SD: track 33.5 -> 0.00 mm, vias 1 -> 0
- net /Mic14/WS: track 33.3 -> 0.00 mm
- net /Mic16/WS: track 33.1 -> 0.00 mm
- net /Mic10/WS: track 32.7 -> 0.00 mm
- net /Mic12/WS: track 32.7 -> 0.00 mm
- net /Mic13/WS: track 32.2 -> 0.00 mm
- net /Mic11/WS: track 31.6 -> 0.00 mm
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- removed copper zone on B.Cu, net GND
- removed copper zone on F.Cu, net GND
- removed copper zone on In1.Cu, net GND
- removed copper zone on In2.Cu, net VDD
Other:
- board size 100 x 100 mm -> 213.1 x 137.7 mm
- board text added: "3.3V"
- board text added: "5V"
- board text added: "Mic1"
- board text added: "Mic10"
- board text added: "Mic11"
- board text added: "Mic12"
- board text added: "Mic13"
- board text added: "Mic14"
- board text added: "Mic15"
- board text added: "Mic16"
- board text added: "Mic2"
- board text added: "Mic3"
- board text added: "Mic4"
- board text added: "Mic5"
- board text added: "Mic6"
- board text added: "Mic7"
- board text added: "Mic8"
- board text added: "Mic9"
- board text removed: "(nc)"
- board text removed: "1"
- board text removed: "1.8V"
- board text removed: "10"
- board text removed: "11"
- board text removed: "12"
- board text removed: "13"
- board text removed: "14"
- board text removed: "15"
- board text removed: "16"
- board text removed: "2"
- board text removed: "3"
- board text removed: "4"
- board text removed: "5"
- board text removed: "6"
- board text removed: "7"
- board text removed: "8"
- board text removed: "9"
- board text removed: "SCK"
- board text removed: "SD"
- board text removed: "WS"

Commit message: pcb: finished routing mic board and ADC board.
 - BOM complete
 - uController pinout configured with CubeMX and re-checked
Parts:
- removed R50, R52: 49.9k, Resistor_SMD:R_0603_1608Metric
- added D11: SMBJ5340BE3/TR13, Diode_SMD:D_SMB, F.Cu at (194.3, 72.6)
- added R10: 100k, Resistor_SMD:R_0603_1608Metric, F.Cu at (178.5, 115.3)
- added R11: 100k, Resistor_SMD:R_0603_1608Metric, F.Cu at (128.8, 107.4)
- added R13: 100k, Resistor_SMD:R_0603_1608Metric, F.Cu at (158.0, 103.9)
- added TP100: Hole_1.5mm, TestPoint:TestPoint_THTPad_D2.0mm_Drill1.0mm, F.Cu at (109.2, 123.2)
- added TP101: Hole_1.5mm, TestPoint:TestPoint_THTPad_D2.0mm_Drill1.0mm, F.Cu at (109.2, 113.5)
- added TP102: Hole_1.5mm, TestPoint:TestPoint_THTPad_D2.0mm_Drill1.0mm, F.Cu at (112.0, 91.9)
- added TP103: Hole_1.5mm, TestPoint:TestPoint_THTPad_D2.0mm_Drill1.0mm, F.Cu at (144.5, 70.4)
- added TP104: Hole_1.5mm, TestPoint:TestPoint_THTPad_D2.0mm_Drill1.0mm, F.Cu at (112.0, 101.3)
- added TP105: Hole_1.5mm, TestPoint:TestPoint_THTPad_D2.0mm_Drill1.0mm, F.Cu at (147.8, 70.4)
- added TP106: Hole_1.5mm, TestPoint:TestPoint_THTPad_D2.0mm_Drill1.0mm, F.Cu at (112.0, 82.5)
- added TP107: Hole_1.5mm, TestPoint:TestPoint_THTPad_D2.0mm_Drill1.0mm, F.Cu at (157.5, 70.4)
- added TP108: Hole_1.5mm, TestPoint:TestPoint_THTPad_D2.0mm_Drill1.0mm, F.Cu at (168.1, 82.1)
- added TP109: Hole_1.5mm, TestPoint:TestPoint_THTPad_D2.0mm_Drill1.0mm, F.Cu at (188.0, 91.2)
- added TP110: Hole_1.5mm, TestPoint:TestPoint_THTPad_D2.0mm_Drill1.0mm, F.Cu at (154.9, 151.6)
- added TP111: Hole_1.5mm, TestPoint:TestPoint_THTPad_D2.0mm_Drill1.0mm, F.Cu at (168.4, 147.1)
- added TP112: Hole_1.5mm, TestPoint:TestPoint_THTPad_D2.0mm_Drill1.0mm, F.Cu at (189.0, 148.8)
- added TP113: Hole_1.5mm, TestPoint:TestPoint_THTPad_D2.0mm_Drill1.0mm, F.Cu at (189.0, 139.4)
- added TP114: Hole_1.5mm, TestPoint:TestPoint_THTPad_D2.0mm_Drill1.0mm, F.Cu at (151.4, 151.7)
- added TP115: Hole_1.5mm, TestPoint:TestPoint_THTPad_D2.0mm_Drill1.0mm, F.Cu at (141.7, 151.7)
- added TP116: Hole_1.5mm, TestPoint:TestPoint_THTPad_D2.0mm_Drill1.0mm, F.Cu at (112.0, 127.8)
- added TP117: Hole_1.5mm, TestPoint:TestPoint_THTPad_D2.0mm_Drill1.0mm, F.Cu at (112.0, 118.1)
- added TP118: 5019, TestPoint:TestPoint_Keystone_5019_Minature, F.Cu at (116.6, 111.3)
- added TP119: Hole_1.5mm, TestPoint:TestPoint_Keystone_5019_Minature, F.Cu at (165.6, 105.7)
- added TP120: Hole_1.5mm, TestPoint:TestPoint_Keystone_5019_Minature, F.Cu at (130.3, 68.3)
- added TP121: Hole_1.5mm, TestPoint:TestPoint_Keystone_5019_Minature, F.Cu at (181.6, 152.7)
- added TP38: Hole_1.5mm, TestPoint:TestPoint_THTPad_D2.0mm_Drill1.0mm, F.Cu at (109.2, 96.5)
- added TP39: Hole_1.5mm, TestPoint:TestPoint_THTPad_D2.0mm_Drill1.0mm, F.Cu at (112.0, 98.0)
- added TP40: Hole_1.5mm, TestPoint:TestPoint_THTPad_D2.0mm_Drill1.0mm, F.Cu at (140.0, 67.6)
- added TP41: Hole_1.5mm, TestPoint:TestPoint_THTPad_D2.0mm_Drill1.0mm, F.Cu at (138.4, 70.4)
- added TP42: Hole_1.5mm, TestPoint:TestPoint_THTPad_D2.0mm_Drill1.0mm, F.Cu at (109.2, 105.9)
- added TP43: Hole_1.5mm, TestPoint:TestPoint_THTPad_D2.0mm_Drill1.0mm, F.Cu at (112.0, 107.4)
- added TP44: Hole_1.5mm, TestPoint:TestPoint_THTPad_D2.0mm_Drill1.0mm, F.Cu at (149.4, 67.6)
- added TP45: Hole_1.5mm, TestPoint:TestPoint_THTPad_D2.0mm_Drill1.0mm, F.Cu at (153.9, 70.4)
- added TP46: Hole_1.5mm, TestPoint:TestPoint_THTPad_D2.0mm_Drill1.0mm, F.Cu at (109.2, 87.1)
- added TP47: Hole_1.5mm, TestPoint:TestPoint_THTPad_D2.0mm_Drill1.0mm, F.Cu at (112.0, 88.6)
- added TP48: Hole_1.5mm, TestPoint:TestPoint_THTPad_D2.0mm_Drill1.0mm, F.Cu at (159.0, 67.6)
- added TP49: Hole_1.5mm, TestPoint:TestPoint_THTPad_D2.0mm_Drill1.0mm, F.Cu at (163.6, 70.4)
- added TP50: Hole_1.5mm, TestPoint:TestPoint_THTPad_D2.0mm_Drill1.0mm, F.Cu at (169.7, 79.2)
- added TP51: Hole_1.5mm, TestPoint:TestPoint_THTPad_D2.0mm_Drill1.0mm, F.Cu at (174.2, 82.0)
- added TP52: Hole_1.5mm, TestPoint:TestPoint_THTPad_D2.0mm_Drill1.0mm, F.Cu at (190.8, 92.7)
- added TP53: Hole_1.5mm, TestPoint:TestPoint_THTPad_D2.0mm_Drill1.0mm, F.Cu at (187.9, 97.3)
- added TP54: Hole_1.5mm, TestPoint:TestPoint_THTPad_D2.0mm_Drill1.0mm, F.Cu at (159.5, 154.4)
- added TP55: Hole_1.5mm, TestPoint:TestPoint_THTPad_D2.0mm_Drill1.0mm, F.Cu at (161.0, 151.6)
- added TP56: Hole_1.5mm, TestPoint:TestPoint_THTPad_D2.0mm_Drill1.0mm, F.Cu at (173.0, 149.9)
- added TP57: Hole_1.5mm, TestPoint:TestPoint_THTPad_D2.0mm_Drill1.0mm, F.Cu at (174.5, 147.1)
- added TP58: Hole_1.5mm, TestPoint:TestPoint_THTPad_D2.0mm_Drill1.0mm, F.Cu at (191.8, 144.3)
- added TP59: Hole_1.5mm, TestPoint:TestPoint_THTPad_D2.0mm_Drill1.0mm, F.Cu at (189.0, 142.7)
- added TP60: Hole_1.5mm, TestPoint:TestPoint_THTPad_D2.0mm_Drill1.0mm, F.Cu at (191.8, 134.9)
- added TP61: Hole_1.5mm, TestPoint:TestPoint_THTPad_D2.0mm_Drill1.0mm, F.Cu at (189.0, 133.3)
- added TP62: Hole_1.5mm, TestPoint:TestPoint_THTPad_D2.0mm_Drill1.0mm, F.Cu at (149.9, 154.4)
- added TP63: Hole_1.5mm, TestPoint:TestPoint_THTPad_D2.0mm_Drill1.0mm, F.Cu at (145.3, 151.6)
- added TP64: Hole_1.5mm, TestPoint:TestPoint_THTPad_D2.0mm_Drill1.0mm, F.Cu at (140.2, 154.4)
- added TP65: Hole_1.5mm, TestPoint:TestPoint_THTPad_D2.0mm_Drill1.0mm, F.Cu at (135.6, 151.6)
- added TP66: Hole_1.5mm, TestPoint:TestPoint_THTPad_D2.0mm_Drill1.0mm, F.Cu at (109.2, 126.2)
- added TP67: Hole_1.5mm, TestPoint:TestPoint_THTPad_D2.0mm_Drill1.0mm, F.Cu at (112.0, 121.7)
- added TP68: Hole_1.5mm, TestPoint:TestPoint_THTPad_D2.0mm_Drill1.0mm, F.Cu at (109.2, 116.6)
- added TP69: Hole_1.5mm, TestPoint:TestPoint_THTPad_D2.0mm_Drill1.0mm, F.Cu at (112.0, 112.0)
- added TP70: Hole_1.5mm, TestPoint:TestPoint_THTPad_D2.0mm_Drill1.0mm, F.Cu at (112.0, 95.0)
- added TP71: Hole_1.5mm, TestPoint:TestPoint_THTPad_D2.0mm_Drill1.0mm, F.Cu at (141.5, 70.4)
- added TP72: Hole_1.5mm, TestPoint:TestPoint_THTPad_D2.0mm_Drill1.0mm, F.Cu at (112.0, 104.4)
- added TP73: Hole_1.5mm, TestPoint:TestPoint_THTPad_D2.0mm_Drill1.0mm, F.Cu at (150.9, 70.4)
- added TP74: Hole_1.5mm, TestPoint:TestPoint_THTPad_D2.0mm_Drill1.0mm, F.Cu at (112.0, 85.6)
- added TP75: Hole_1.5mm, TestPoint:TestPoint_THTPad_D2.0mm_Drill1.0mm, F.Cu at (160.6, 70.4)
- added TP76: Hole_1.5mm, TestPoint:TestPoint_THTPad_D2.0mm_Drill1.0mm, F.Cu at (171.2, 82.0)
- added TP77: Hole_1.5mm, TestPoint:TestPoint_THTPad_D2.0mm_Drill1.0mm, F.Cu at (187.9, 94.2)
- added TP78: Hole_1.5mm, TestPoint:TestPoint_THTPad_D2.0mm_Drill1.0mm, F.Cu at (158.0, 151.6)
- added TP79: Hole_1.5mm, TestPoint:TestPoint_THTPad_D2.0mm_Drill1.0mm, F.Cu at (171.5, 147.1)
- added TP80: Hole_1.5mm, TestPoint:TestPoint_THTPad_D2.0mm_Drill1.0mm, F.Cu at (189.0, 145.8)
- added TP81: Hole_1.5mm, TestPoint:TestPoint_THTPad_D2.0mm_Drill1.0mm, F.Cu at (189.0, 136.4)
- added TP82: Hole_1.5mm, TestPoint:TestPoint_THTPad_D2.0mm_Drill1.0mm, F.Cu at (148.3, 151.6)
- added TP83: Hole_1.5mm, TestPoint:TestPoint_THTPad_D2.0mm_Drill1.0mm, F.Cu at (138.7, 151.6)
- added TP84: Hole_1.5mm, TestPoint:TestPoint_THTPad_D2.0mm_Drill1.0mm, F.Cu at (112.0, 124.7)
- added TP85: Hole_1.5mm, TestPoint:TestPoint_THTPad_D2.0mm_Drill1.0mm, F.Cu at (112.0, 115.1)
- added TP86: Hole_1.5mm, TestPoint:TestPoint_THTPad_D2.0mm_Drill1.0mm, F.Cu at (109.2, 93.5)
- added TP87: Hole_1.5mm, TestPoint:TestPoint_THTPad_D2.0mm_Drill1.0mm, F.Cu at (143.0, 67.6)
- added TP88: Hole_1.5mm, TestPoint:TestPoint_THTPad_D2.0mm_Drill1.0mm, F.Cu at (109.2, 102.9)
- added TP89: Hole_1.5mm, TestPoint:TestPoint_THTPad_D2.0mm_Drill1.0mm, F.Cu at (152.4, 67.6)
- added TP90: Hole_1.5mm, TestPoint:TestPoint_THTPad_D2.0mm_Drill1.0mm, F.Cu at (109.2, 84.1)
- added TP91: Hole_1.5mm, TestPoint:TestPoint_THTPad_D2.0mm_Drill1.0mm, F.Cu at (162.1, 67.6)
- added TP92: Hole_1.5mm, TestPoint:TestPoint_THTPad_D2.0mm_Drill1.0mm, F.Cu at (172.7, 79.2)
- added TP93: Hole_1.5mm, TestPoint:TestPoint_THTPad_D2.0mm_Drill1.0mm, F.Cu at (190.8, 95.8)
- added TP94: Hole_1.5mm, TestPoint:TestPoint_THTPad_D2.0mm_Drill1.0mm, F.Cu at (156.5, 154.4)
- added TP95: Hole_1.5mm, TestPoint:TestPoint_THTPad_D2.0mm_Drill1.0mm, F.Cu at (169.9, 149.9)
- added TP96: Hole_1.5mm, TestPoint:TestPoint_THTPad_D2.0mm_Drill1.0mm, F.Cu at (191.8, 147.3)
- added TP97: Hole_1.5mm, TestPoint:TestPoint_THTPad_D2.0mm_Drill1.0mm, F.Cu at (191.8, 137.9)
- added TP98: Hole_1.5mm, TestPoint:TestPoint_THTPad_D2.0mm_Drill1.0mm, F.Cu at (146.8, 154.4)
- added TP99: Hole_1.5mm, TestPoint:TestPoint_THTPad_D2.0mm_Drill1.0mm, F.Cu at (137.2, 154.4)
- C1, C10, C2, C3, C4, C5, C6, C67, C68, C69, C7, C70, C71, C72, C73, C74, C75, C76, C8, C9, JP1, JP2: moved to B.Cu
- C16, C77: value 1uF -> 10uF; footprint Capacitor_SMD:C_0603_1608Metric -> Capacitor_SMD:C_0805_2012Metric
- moved R135 135.8 mm to (103.1, 132.8)
- moved R136 135.8 mm to (103.1, 136.1)
- moved R138 135.8 mm to (103.1, 142.2)
- moved JP5 135.8 mm to (110.0, 147.8)
- moved D6 135.8 mm to (106.5, 142.0)
- moved D3 135.8 mm to (106.5, 132.6)
- moved D4 135.8 mm to (106.5, 135.9)
- moved R139 135.8 mm to (103.1, 145.3)
- moved JP10 135.8 mm to (109.9, 132.6)
- moved R137 135.8 mm to (103.2, 139.2)
- moved JP4 135.8 mm to (110.0, 150.9)
- moved D5 135.8 mm to (106.6, 138.9)
- moved D7 135.8 mm to (106.5, 145.0)
- moved JP7 135.7 mm to (110.0, 141.7)
- moved JP9 135.7 mm to (109.9, 135.6)
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Connections:
- U1 pad 5: (no net) -> unconnected-(U1-NC-Pad5)
- U1 pad 7: (no net) -> unconnected-(U1-NC-Pad7)
- U1 pad 9: (no net) -> unconnected-(U1-EP-Pad9)
- U34 pad 12: unconnected-(U34D-A4-Pad12) -> GND
- U34 pad 15: (no net) -> GND
- U5 pad 1: unconnected-(U5-PC10-Pad1) -> /uController/~{PButton1}
- U5 pad 101: unconnected-(U5-PB5-Pad101) -> /uController/SPI1_MOSI_uC
- U5 pad 113: unconnected-(U5-PD13-Pad113) -> /uController/SPI1_~{CS2}_uC
- U5 pad 140: /DRDY -> unconnected-(U5-PG5-Pad140)
- U5 pad 141: /uController/GPIO_~{START}_uC -> unconnected-(U5-PG4-Pad141)
- U5 pad 2: unconnected-(U5-PC11-Pad2) -> /uController/~{PButton2}
- U5 pad 38: unconnected-(U5-PC0-Pad38) -> /DRDY
- U5 pad 39: /uController/LED5_uC -> unconnected-(U5-PD4-Pad39)
- U5 pad 4: /uController/LED3_uC -> unconnected-(U5-PD2-Pad4)
- U5 pad 40: /uController/LED4_uC -> unconnected-(U5-PD3-Pad40)
- U5 pad 41: /uController/LED6_uC -> unconnected-(U5-PD5-Pad41)
- U5 pad 43: /uController/LED7_uC -> unconnected-(U5-PD6-Pad43)
- U5 pad 45: /uController/SPI1_MOSI_uC -> unconnected-(U5-PD7-Pad45)
- U5 pad 55: /uController/LED2_uC -> /uController/LED8_uC
- U5 pad 57: /uController/LED1_uC -> /uController/LED7_uC
- U5 pad 58: unconnected-(U5-PG1-Pad58) -> /uController/LED6_uC
- U5 pad 59: unconnected-(U5-PG0-Pad59) -> /uController/LED5_uC
- U5 pad 61: unconnected-(U5-PE1-Pad61) -> /uController/LED_DevLD2
- U5 pad 62: unconnected-(U5-PE6-Pad62) -> /uController/LED4_uC
- U5 pad 63: /uController/LED8_uC -> /uController/LED3_uC
- U5 pad 64: unconnected-(U5-PG15-Pad64) -> /uController/LED2_uC
- U5 pad 65: unconnected-(U5-PG12-Pad65) -> /uController/LED1_uC
- U5 pad 66: /uController/SPI1_~{CS2}_uC -> unconnected-(U5-PG10-Pad66)
- U5 pad 94: /uController/~{PButton2} -> /uController/GPIO_~{START}_uC
- U5 pad 96: /uController/~{PButton1} -> unconnected-(U5-PB1-Pad96)
- U6 pad 26: /ADC1 AD7768/DOUT7 -> /ADC1 AD7768/DOUT6
- U6 pad 27: /ADC1 AD7768/DOUT6 -> /ADC1 AD7768/DOUT7
Routing:
- net +3.3VA: track 0.00 -> 451.3 mm, vias 0 -> 1
- net +3.3V: track 0.00 -> 203.5 mm, vias 0 -> 14
- net GND: track 0.00 -> 161.7 mm, vias 0 -> 78
- net +5VA: track 0.00 -> 118.9 mm, vias 0 -> 5
- net /uController/V_{IN}: track 0.00 -> 105.0 mm, vias 0 -> 1
- net /V_{REF}: track 0.00 -> 95.0 mm, vias 0 -> 3
- net /V_{IN}: track 0.00 -> 89.9 mm
- net /SPI1_SCLK: track 0.00 -> 80.3 mm, vias 0 -> 3
- net /SPI1_MISO: track 0.00 -> 76.4 mm, vias 0 -> 3
- net /uController/SPI2_SCLK_buff: track 0.00 -> 72.8 mm, vias 0 -> 2
- net /SPI1_MOSI: track 0.00 -> 54.9 mm, vias 0 -> 3
- net /DRDY: track 0.00 -> 43.8 mm, vias 0 -> 2
- net /ADC1 AD7768/DCLK: track 0.00 -> 37.5 mm, vias 0 -> 2
- net /ADC1 AD7768/~{SYNC_IN}: track 0.00 -> 35.0 mm, vias 0 -> 2
- net /ADC1 AD7768/~{START}: track 0.00 -> 30.8 mm
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- added copper zone on In2.Cu, net +3.3V
- added copper zone on B.Cu, net GND
- added copper zone on F.Cu, net GND
- added copper zone on In1.Cu, net GND
Other:
- board size 213.1 x 137.7 mm -> 100 x 100 mm
- board text added: "+|-|S G|V"
- board text added: "Ethernet Jack"
- board text added: "JBRRY SoundCompass Mic eval board v202405xx"
- board text added: "ST-Link"
- board text added: "S|-|+ G|V"
- board text added: "V_{IN}: 5.2-6.5V"
- board text added: "Vin Gnd"
- board text removed: "3-5V In"
- board text removed: "Gnd"
- board text removed: "jbrry SoundCompass Mic eval board v202402xx"

Commit message: pcb: ordered PCB's and BOM! RevA and v240506
Parts:
- removed H1, H2, H3: MountingHole, MountingHole:MountingHole_3.2mm_M3
Other:
- board text added: "JBRRY SoundCompass Mic Test Board v20240506"
- board text removed: "JBRRY SoundCompass Mic eval board v202405xx"
