File: sch/mic-test-board/Power.kicad_sch (KiCad schematic)
At the start: 27 parts, among them U22 LP5912-5.0DRV, U23 LP5912-3.3DRV, U24 LP5912-3.3DRV

Commit message: pcb: commit before large routing effort
 - schematic refactor to split preamps to each mic board
 - Mic board and main board are placed
 - no tracks laid
 - critical parts selected
Parts:
- removed D1, D2: LED_Small_Filled, LED_SMD:LED_0805_2012Metric, symbol Device:LED_Small_Filled
- removed R33, R4: 0R, Resistor_SMD:R_0603_1608Metric, symbol Device:R_Small
- added J2: Conn_01x03, Connector_PinHeader_2.54mm:PinHeader_1x02_P2.54mm_Vertical, symbol Connector_Generic:Conn_01x02
- C59, C60, C61, C62, C63, C64: footprint (none) -> Capacitor_SMD:C_0603_1608Metric
- JP18: footprint (none) -> Jumper:SolderJumper-3_P1.3mm_Open_RoundedPad1.0x1.5mm_NumberLabels
- JP19: footprint (none) -> ~
- R26, R28, R29, R31, R32, R34: footprint (none) -> Resistor_SMD:R_0603_1608Metric
- TP10, TP11, TP12, TP7, TP8, TP9: footprint (none) -> TestPoint:TestPoint_Pad_D1.0mm
Connections:
- net +3.3V: no longer C62.1, JP18.3 (B), R31.2, U24.1 (OUT)
- net +3.3VA: no longer JP18.2 (C)
- net +5VA: no longer C59.1, R29.2, U22.1 (OUT)
- new net 3.3V: C62.1, JP18.3 (B), R31.2, U24.1 (OUT)
- new net 3.3VA: JP18.2 (C)
- new net 5VA: C59.1, R29.2, U22.1 (OUT)
- no-connect marks 0 -> 3
Other:
- note added: "LDO"
- note added: "Mics and preamps are off the main board"
- note added: "Nucleo Dev board"
- note added: "Terminal"
- note added: "x16"
- note removed: "The 3.3V will power the ADC digital section and the mics. If the 3.3V rail is too noisy, and the mic PSR is not good enough, there is another 3.3V LDO to swap in."
- note removed: "Vf = 1.85V"
- company: (none) -> Josh Berry
- title: (none) -> Sound Compass POC
- moved on the sheet: C59, C60, C61, C62, C63, C64, JP18, R26, R28, R29, R31, R32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

Commit message: pcb: finished routing mic board and ADC board.
 - BOM complete
 - uController pinout configured with CubeMX and re-checked
Parts:
- C59, C60, C61, C62, C63, C64: Manufacturer (none) -> YAGEO; Part Number (none) -> CC0603KRX7R7BB105; Supplier (none) -> Digi-Key; Supplier Number (none) -> 311-1446-1-ND
- J2: footprint Connector_PinHeader_2.54mm:PinHeader_1x02_P2.54mm_Vertical -> ~; now not fitted
- JP18, JP19, TP10, TP11, TP12, TP7, TP8, TP9: now not fitted
- R26, R28: Manufacturer (none) -> Stackpole Electronics Inc; Part Number (none) -> RMCF0603ZT0R00; Supplier (none) -> Digi-Key; Supplier Number (none) -> RMCF0603ZT0R00CT-ND
- R29, R31: Manufacturer (none) -> YAGEO; Part Number (none) -> RC0603FR-07100KL; Supplier (none) -> Digi-Key; Supplier Number (none) -> 311-100KHRCT-ND
- U22: Manufacturer (none) -> Texas Instruments; Part Number (none) -> LP5912-5.0DRVR; Supplier (none) -> Digi-Key; Supplier Number (none) -> 296-53182-1-ND
- U24: Manufacturer (none) -> Texas Instruments; Part Number (none) -> LP5912-3.3DRVR; Supplier (none) -> Digi-Key; Supplier Number (none) -> 296-47214-1-ND
Other:
- note added: "x2"

Commit message: pcb: ordered PCB's and BOM! RevA and v240506
Parts:
- J2: value Conn_01x03 -> Conn_01x02; now fitted
- JP18, TP10, TP7, TP8, TP9: now fitted; now left out of the parts list
- JP19: now fitted
- R32: Manufacturer (none) -> Stackpole Electronics Inc; Part Number (none) -> RMCF0603ZT0R00; Supplier (none) -> Digi-Key; Supplier Number (none) -> RMCF0603ZT0R00CT-ND
- R34: Manufacturer (none) -> YAGEO; Part Number (none) -> RC0603FR-07100KL; Supplier (none) -> Digi-Key; Supplier Number (none) -> 311-100KHRCT-ND
- TP11, TP12: now left out of the parts list
- U23: Manufacturer (none) -> Texas Instruments; Part Number (none) -> LP5912-3.3DRVR; Supplier (none) -> Digi-Key; Supplier Number (none) -> 296-47214-1-ND
